Commit message: [description] Fixed naming error from old package name

File: description/xacro/hokuyo.xacro (robot description, xacro)
@@ -1,7 +1,7 @@
 <?xml version="1.0"?>
 <root xmlns:sensor="http://playerstage.sourceforge.net/gazebo/xmlschema/#sensor"
-       xmlns:controller="http://playerstage.sourceforge.net/gazebo/xmlschema/#controller"
-       xmlns:interface="http://playerstage.sourceforge.net/gazebo/xmlschema/#interface"
-       xmlns:xacro="http://ros.org/wiki/xacro">
+      xmlns:controller="http://playerstage.sourceforge.net/gazebo/xmlschema/#controller"
+      xmlns:interface="http://playerstage.sourceforge.net/gazebo/xmlschema/#interface"
+      xmlns:xacro="http://ros.org/wiki/xacro">
     <xacro:macro name="hokuyo" params="name parent *origin namespace ros_topic update_rate min_angle max_angle">
         <joint name="${name}_joint" type="fixed">
@@ -20,5 +20,5 @@
                 <origin xyz="0 0 0" rpy="0 0 0"/>
                 <geometry>
-                    <mesh filename="package://ropod_description/meshes/hokuyo.dae"/>
+                    <mesh filename="package://ropod_sim/description/meshes/hokuyo.dae"/>
                 </geometry>
             </visual>

File: description/xacro/ropod.xacro (robot description, xacro)
@@ -16,5 +16,5 @@
     <xacro:property name="inertia_base" value="0.5" />
     <xacro:property name="inertia_wheels" value="0.001" />
-    <xacro:include filename="$(find ropod_description)/xacro/hokuyo.xacro" />
+    <xacro:include filename="$(find ropod_sim)/description/xacro/hokuyo.xacro" />
     <material name="silver">
         <color rgba="0.6 0.6 0.6 1.0"/>
