Commit message: [description] Removed friction of wheels with the floor

File: description/xacro/ropod.xacro (robot description, xacro)
@@ -53,4 +53,6 @@
         </link>
         <gazebo reference="${name}_link">
+            <mu1>0.0</mu1>
+            <mu2>0.0</mu2>
             <material>Gazebo/Black</material>
         </gazebo>
@@ -141,5 +143,5 @@
         <collision>
             <geometry>
-                <box size='0.2 0.3 0.1'/>
+                <box size='0.01 0.01 0.01'/>
             </geometry>
         </collision>

Commit message: [description][plugin] Removed docking info in plugin

File: description/xacro/ropod.xacro (robot description, xacro)
@@ -1,12 +1,6 @@
 <?xml version='1.0'?>
-<robot xmlns:sensor="http://playerstage.sourceforge.net/gazebo/xmlschema/#sensor"
-       xmlns:controller="http://playerstage.sourceforge.net/gazebo/xmlschema/#controller"
-       xmlns:interface="http://playerstage.sourceforge.net/gazebo/xmlschema/#interface"
-       xmlns:xacro="http://ros.org/wiki/xacro"
-       name="ropod" >
+<robot xmlns:xacro="http://ros.org/wiki/xacro" name="ropod" >
     <xacro:property name="namespace" value="$(arg namespace)"/>
     <xacro:arg name="namespace" default="ropod"/>
-    <xacro:property name="cart_length" value="$(arg cart_length)"/>
-    <xacro:arg name="cart_length" default="1.1"/>
     <xacro:property name="base_length" value="0.6" />
     <xacro:property name="base_thickness" value="0.1" />
@@ -58,8 +52,8 @@
         </gazebo>
     </xacro:macro>
-    <link name='base_link_ground' />
+    <link name='base_link' />
     <joint name='base_body_joint' type='fixed'>
         <origin xyz='0.0 0.0 ${wheel_radius*2 + base_thickness*0.5}' rpy='0 0 0'/>
-        <parent link='base_link_ground'/>
+        <parent link='base_link'/>
         <child link='base_body_link'/>
     </joint>
@@ -118,10 +112,8 @@
         <plugin name="${namespace}_controller" filename="libropod_control_plugin.so">
             <commandTopic>/${namespace}/cmd_vel</commandTopic>
-            <dockTopic>/${namespace}/dock</dockTopic>
             <odometryTopic>/${namespace}/odom</odometryTopic>
             <odometryFrame>/${namespace}/odom</odometryFrame>
             <odometryRate>20.0</odometryRate>
             <robotBaseFrame>/${namespace}/base_link</robotBaseFrame>
-            <dockedBaseLinkOffset>${cart_length}</dockedBaseLinkOffset>
         </plugin>
     </gazebo>

Commit message: [description][ropod] Added realsense_d435 camera to front of robot

File: description/xacro/ropod.xacro (robot description, xacro)
@@ -11,4 +11,5 @@
     <xacro:property name="inertia_wheels" value="0.001" />
     <xacro:include filename="$(find ropod_sim)/description/xacro/hokuyo.xacro" />
+    <xacro:include filename="$(find ropod_sim)/description/xacro/realsense_d435.xacro" />
     <material name="silver">
         <color rgba="0.6 0.6 0.6 1.0"/>
@@ -129,4 +130,7 @@
         <origin xyz="0.25 0.0 0.08" rpy="0 0 0"/>
     </xacro:hokuyo>
+    <xacro:realsense_d435 name="realsense_front" parent="base_link" namespace="${namespace}">
+        <origin xyz="0.3 0.0 0.15" rpy="0.0 0.0 0.0"/>
+    </xacro:realsense_d435>
     <!-- ====================== -->
     <!-- HOLONOMIC DRIVE PLUGIN -->

Commit message: [description][ropod] Added torso camera

File: description/xacro/ropod.xacro (robot description, xacro)
@@ -130,6 +130,12 @@
         <origin xyz="0.25 0.0 0.08" rpy="0 0 0"/>
     </xacro:hokuyo>
+    <!-- ========= -->
+    <!-- 3D CAMERA -->
+    <!-- ========= -->
     <xacro:realsense_d435 name="realsense_front" parent="base_link" namespace="${namespace}">
         <origin xyz="0.3 0.0 0.15" rpy="0.0 0.0 0.0"/>
+    </xacro:realsense_d435>
+    <xacro:realsense_d435 name="realsense_torso" parent="base_link" namespace="${namespace}">
+        <origin xyz="-0.1 0.0 1.0" rpy="0.0 1.0 ${pi}"/>
     </xacro:realsense_d435>
     <!-- ====================== -->
