Commit message: [ros] Updated cart_manager and dock_manager to not use cart_length

File: description/xacro/mobidik.xacro (robot description, xacro)
@@ -1,8 +1,4 @@
 <?xml version='1.0'?>
-<robot xmlns:sensor="http://playerstage.sourceforge.net/gazebo/xmlschema/#sensor"
-       xmlns:controller="http://playerstage.sourceforge.net/gazebo/xmlschema/#controller"
-       xmlns:interface="http://playerstage.sourceforge.net/gazebo/xmlschema/#interface"
-       xmlns:xacro="http://ros.org/wiki/xacro"
-       name="mobidik" >
+<robot xmlns:xacro="http://ros.org/wiki/xacro" name="mobidik" >
     <xacro:arg name="namespace" default="ropod"/>
     <xacro:property name="namespace" value="$(arg namespace)"/>
@@ -107,4 +103,27 @@
         <origin xyz='${base_length*0.5 - wheel_radius} ${-base_width*0.5 + wheel_radius} ${-base_thickness*0.5 - wheel_radius}' rpy='0 0 0'/>
     </xacro:cart_wheel>
+    <!-- ======= -->
+    <!-- GRIPPER -->
+    <!-- ======= -->
+    <joint name='gripping_joint' type='fixed'>
+        <origin xyz='${base_length*0.5} 0.0 ${wheel_radius*2}' rpy='0 0 0'/>
+        <parent link='base_link'/>
+        <child link='gripping_link'/>
+    </joint>
+    <link name='gripping_link'>
+        <visual>
+            <geometry>
+                <box size="${0.01} ${0.01} ${0.01}"/>
+            </geometry>
+            <origin xyz='0.0 0.0 0.0' rpy='0.0 0.0 0.0' />
+            <material name="red"/>
+        </visual>
+        <collision>
+            <geometry>
+                <box size="${0.01} ${0.01} ${0.01}"/>
+            </geometry>
+            <origin xyz='0.0 0.0 0.0' rpy='0.0 0.0 0.0' />
+        </collision>
+    </link>
     <!-- ===== -->
     <!-- CARGO -->

File: description/xacro/ropod.xacro (robot description, xacro)
@@ -99,4 +99,27 @@
         <origin xyz='${base_length*0.5 - wheel_radius} ${-base_length*0.5 + wheel_radius} ${-base_thickness*0.5 - wheel_radius}' rpy='0 0 0'/>
     </xacro:ropod_wheel>
+    <!-- ======= -->
+    <!-- GRIPPER -->
+    <!-- ======= -->
+    <joint name='gripper_joint' type='fixed'>
+        <origin xyz='${-base_length*0.5} 0.0 ${wheel_radius*2}' rpy='0 0 0'/>
+        <parent link='base_link'/>
+        <child link='gripper_link'/>
+    </joint>
+    <link name='gripper_link'>
+        <visual>
+            <geometry>
+                <box size="${0.01} ${0.01} ${0.01}"/>
+            </geometry>
+            <origin xyz='0.0 0.0 0.0' rpy='0.0 0.0 0.0' />
+            <material name="silver"/>
+        </visual>
+        <collision>
+            <geometry>
+                <box size="${0.01} ${0.01} ${0.01}"/>
+            </geometry>
+            <origin xyz='0.0 0.0 0.0' rpy='0.0 0.0 0.0' />
+        </collision>
+    </link>
     <!-- ===== -->
     <!-- LASER -->

Commit message: [description][mobidik] Increased length of cargo

File: description/xacro/mobidik.xacro (robot description, xacro)
@@ -6,5 +6,5 @@
     <xacro:property name="base_width" value="0.8" />
     <xacro:property name="base_thickness" value="0.1" />
-    <xacro:property name="cargo_length" value="0.7" />
+    <xacro:property name="cargo_length" value="1.0" />
     <xacro:property name="cargo_width" value="0.7" />
     <xacro:property name="cargo_height" value="1.0" />

Commit message: [description][mobidik] Added aruco markers to cart

File: description/xacro/mobidik.xacro (robot description, xacro)
@@ -1,3 +1,3 @@
-<?xml version='1.0'?>
+<?xml version="1.0"?>
 <robot xmlns:xacro="http://ros.org/wiki/xacro" name="mobidik" >
     <xacro:arg name="namespace" default="ropod"/>
@@ -10,4 +10,5 @@
     <xacro:property name="cargo_height" value="1.0" />
     <xacro:property name="wheel_radius" value="0.04" />
+    <xacro:property name="marker_length" value="0.2" />
     <xacro:property name="wheel_mass" value="1.0" />
     <xacro:property name="base_mass" value="8.0" />
@@ -22,4 +23,7 @@
     <material name="brown">
         <color rgba="0.8 0.52 0.25 1.0"/>
+    </material>
+    <material name="white">
+        <color rgba="1.0 1.0 1.0 1.0"/>
     </material>
     <xacro:macro name="sphere_inertia" params="mass radius">
@@ -56,16 +60,39 @@
         </gazebo>
     </xacro:macro>
-    <link name='base_link' />
-    <joint name='base_body_joint' type='fixed'>
-        <origin xyz='0.0 0.0 ${wheel_radius*2 + base_thickness*0.5}' rpy='0 0 0'/>
-        <parent link='base_link'/>
-        <child link='base_body_link'/>
+    <xacro:macro name="aruco_marker" params="name parent *origin length gazebo_material_name">
+        <joint name="${name}_joint" type="fixed">
+            <xacro:insert_block name="origin" />
+            <parent link="${parent}_link"/>
+            <child link="${name}_link"/>
+        </joint>
+        <link name="${name}_link">
+            <visual>
+                <geometry>
+                    <box size="0.0001 ${marker_length} ${marker_length}"/>
+                </geometry>
+                <material name="white"/>
+            </visual>
+            <collision>
+                <geometry>
+                    <box size="0.0001 ${marker_length} ${marker_length}"/>
+                </geometry>
+            </collision>
+        </link>
+        <gazebo reference="${name}_link">
+            <material>${gazebo_material_name}</material>
+        </gazebo>
+    </xacro:macro>
+    <link name="base_link" />
+    <joint name="base_body_joint" type="fixed">
+        <origin xyz="0.0 0.0 ${wheel_radius*2 + base_thickness*0.5}" rpy="0 0 0"/>
+        <parent link="base_link"/>
+        <child link="base_body_link"/>
     </joint>
-    <link name='base_body_link'>
+    <link name="base_body_link">
         <visual>
             <geometry>
                 <box size="${base_length} ${base_width} ${base_thickness}"/>
             </geometry>
-            <origin xyz='0.0 0.0 0.0' rpy='0.0 0.0 0.0' />
+            <origin xyz="0.0 0.0 0.0" rpy="0.0 0.0 0.0" />
             <material name="red"/>
         </visual>
@@ -74,5 +101,5 @@
                 <box size="${base_length} ${base_width} ${base_thickness}"/>
             </geometry>
-            <origin xyz='0.0 0.0 0.0' rpy='0.0 0.0 0.0' />
+            <origin xyz="0.0 0.0 0.0" rpy="0.0 0.0 0.0" />
         </collision>
         <inertial>
@@ -89,32 +116,32 @@
     <xacro:cart_wheel name="left_rear_wheel" parent="base_body" mass="${wheel_mass}"
                        radius="${wheel_radius}" material_name="black">
-        <origin xyz='${-base_length*0.5 + wheel_radius} ${base_width*0.5 - wheel_radius} ${-base_thickness*0.5 - wheel_radius}' rpy='0 0 0'/>
+        <origin xyz="${-base_length*0.5 + wheel_radius} ${base_width*0.5 - wheel_radius} ${-base_thickness*0.5 - wheel_radius}" rpy="0 0 0"/>
     </xacro:cart_wheel>
     <xacro:cart_wheel name="right_rear_wheel" parent="base_body" mass="${wheel_mass}"
                        radius="${wheel_radius}" material_name="black">
-        <origin xyz='${-base_length*0.5 + wheel_radius} ${-base_width*0.5 + wheel_radius} ${-base_thickness*0.5 - wheel_radius}' rpy='0 0 0'/>
+        <origin xyz="${-base_length*0.5 + wheel_radius} ${-base_width*0.5 + wheel_radius} ${-base_thickness*0.5 - wheel_radius}" rpy="0 0 0"/>
     </xacro:cart_wheel>
     <xacro:cart_wheel name="left_front_wheel" parent="base_body" mass="${wheel_mass}"
                        radius="${wheel_radius}" material_name="black">
-        <origin xyz='${base_length*0.5 - wheel_radius} ${base_width*0.5 - wheel_radius} ${-base_thickness*0.5 - wheel_radius}' rpy='0 0 0'/>
+        <origin xyz="${base_length*0.5 - wheel_radius} ${base_width*0.5 - wheel_radius} ${-base_thickness*0.5 - wheel_radius}" rpy="0 0 0"/>
     </xacro:cart_wheel>
     <xacro:cart_wheel name="right_front_wheel" parent="base_body" mass="${wheel_mass}"
                        radius="${wheel_radius}" material_name="black">
-        <origin xyz='${base_length*0.5 - wheel_radius} ${-base_width*0.5 + wheel_radius} ${-base_thickness*0.5 - wheel_radius}' rpy='0 0 0'/>
+        <origin xyz="${base_length*0.5 - wheel_radius} ${-base_width*0.5 + wheel_radius} ${-base_thickness*0.5 - wheel_radius}" rpy="0 0 0"/>
     </xacro:cart_wheel>
     <!-- ======= -->
     <!-- GRIPPER -->
     <!-- ======= -->
-    <joint name='gripping_joint' type='fixed'>
-        <origin xyz='${base_length*0.5} 0.0 ${wheel_radius*2}' rpy='0 0 0'/>
-        <parent link='base_link'/>
-        <child link='gripping_link'/>
+    <joint name="gripping_joint" type="fixed">
+        <origin xyz="${base_length*0.5} 0.0 ${wheel_radius*2}" rpy="0 0 0"/>
+        <parent link="base_link"/>
+        <child link="gripping_link"/>
     </joint>
-    <link name='gripping_link'>
+    <link name="gripping_link">
         <visual>
             <geometry>
                 <box size="${0.01} ${0.01} ${0.01}"/>
             </geometry>
-            <origin xyz='0.0 0.0 0.0' rpy='0.0 0.0 0.0' />
+            <origin xyz="0.0 0.0 0.0" rpy="0.0 0.0 0.0" />
             <material name="red"/>
         </visual>
@@ -123,5 +150,5 @@
                 <box size="${0.01} ${0.01} ${0.01}"/>
             </geometry>
-            <origin xyz='0.0 0.0 0.0' rpy='0.0 0.0 0.0' />
+            <origin xyz="0.0 0.0 0.0" rpy="0.0 0.0 0.0" />
         </collision>
     </link>
@@ -129,13 +156,13 @@
     <!-- CARGO -->
     <!-- ===== -->
-    <joint name='cargo_joint' type='fixed'>
-        <origin xyz='0.0 0.0 ${cargo_height*0.5 + base_thickness*0.5}' rpy='0 0 0'/>
-        <parent link='base_body_link'/>
-        <child link='cargo_link'/>
+    <joint name="cargo_joint" type="fixed">
+        <origin xyz="0.0 0.0 ${cargo_height*0.5 + base_thickness*0.5}" rpy="0 0 0"/>
+        <parent link="base_body_link"/>
+        <child link="cargo_link"/>
     </joint>
-    <link name='cargo_link'>
+    <link name="cargo_link">
         <visual>
             <geometry>
-                <box size='${cargo_length} ${cargo_width} ${cargo_height}'/>
+                <box size="${cargo_length} ${cargo_width} ${cargo_height}"/>
             </geometry>
             <material name="brown"/>
@@ -143,5 +170,5 @@
         <collision>
             <geometry>
-                <box size='${cargo_length} ${cargo_width} ${cargo_height}'/>
+                <box size="${cargo_length} ${cargo_width} ${cargo_height}"/>
             </geometry>
         </collision>
@@ -150,3 +177,18 @@
         <material>Gazebo/WoodPallet</material>
     </gazebo>
+    <!-- ============= -->
+    <!-- ARUCO MARKERS -->
+    <!-- ============= -->
+    <xacro:aruco_marker name="front_aruco" parent="base" length="${marker_length}" gazebo_material_name="Marker0">
+        <origin xyz="${(cargo_length*0.5) + 0.01} 0.0 ${wheel_radius*2 + base_thickness + marker_length*0.5 + 0.05}" rpy="0 0 0"/>
+    </xacro:aruco_marker>
+    <xacro:aruco_marker name="left_aruco" parent="base" length="${marker_length}" gazebo_material_name="Marker1">
+        <origin xyz="0.0 ${(cargo_width*0.5) + 0.01} ${wheel_radius*2 + base_thickness + marker_length*0.5 + 0.05}" rpy="0 0 ${pi/2}"/>
+    </xacro:aruco_marker>
+    <xacro:aruco_marker name="rear_aruco" parent="base" length="${marker_length}" gazebo_material_name="Marker2">
+        <origin xyz="${-(cargo_length*0.5) - 0.01} 0.0 ${wheel_radius*2 + base_thickness + marker_length*0.5 + 0.05}" rpy="0 0 ${pi}"/>
+    </xacro:aruco_marker>
+    <xacro:aruco_marker name="right_aruco" parent="base" length="${marker_length}" gazebo_material_name="Marker3">
+        <origin xyz="0.0 ${-(cargo_width*0.5) - 0.01} ${wheel_radius*2 + base_thickness + marker_length*0.5 + 0.05}" rpy="0 0 ${-pi/2}"/>
+    </xacro:aruco_marker>
 </robot>

File: description/xacro/ropod.xacro (robot description, xacro)
@@ -1,3 +1,3 @@
-<?xml version='1.0'?>
+<?xml version="1.0"?>
 <robot xmlns:xacro="http://ros.org/wiki/xacro" name="ropod" >
     <xacro:property name="namespace" value="$(arg namespace)"/>
@@ -52,16 +52,16 @@
         </gazebo>
     </xacro:macro>
-    <link name='base_link' />
-    <joint name='base_body_joint' type='fixed'>
-        <origin xyz='0.0 0.0 ${wheel_radius*2 + base_thickness*0.5}' rpy='0 0 0'/>
-        <parent link='base_link'/>
-        <child link='base_body_link'/>
+    <link name="base_link" />
+    <joint name="base_body_joint" type="fixed">
+        <origin xyz="0.0 0.0 ${wheel_radius*2 + base_thickness*0.5}" rpy="0 0 0"/>
+        <parent link="base_link"/>
+        <child link="base_body_link"/>
     </joint>
-    <link name='base_body_link'>
+    <link name="base_body_link">
         <visual>
             <geometry>
                 <box size="${base_length} ${base_length} ${base_thickness}"/>
             </geometry>
-            <origin xyz='0.0 0.0 0.0' rpy='0.0 0.0 0.0' />
+            <origin xyz="0.0 0.0 0.0" rpy="0.0 0.0 0.0" />
             <material name="silver"/>
         </visual>
@@ -70,5 +70,5 @@
                 <box size="${base_length} ${base_length} ${base_thickness}"/>
             </geometry>
-            <origin xyz='0.0 0.0 0.0' rpy='0.0 0.0 0.0' />
+            <origin xyz="0.0 0.0 0.0" rpy="0.0 0.0 0.0" />
         </collision>
         <inertial>
@@ -85,32 +85,32 @@
     <xacro:ropod_wheel name="left_rear_wheel" parent="base_body" mass="${wheel_mass}"
                        radius="${wheel_radius}" material_name="black">
-        <origin xyz='${-base_length*0.5 + wheel_radius} ${base_length*0.5 - wheel_radius} ${-base_thickness*0.5 - wheel_radius}' rpy='0 0 0'/>
+        <origin xyz="${-base_length*0.5 + wheel_radius} ${base_length*0.5 - wheel_radius} ${-base_thickness*0.5 - wheel_radius}" rpy="0 0 0"/>
     </xacro:ropod_wheel>
     <xacro:ropod_wheel name="right_rear_wheel" parent="base_body" mass="${wheel_mass}"
                        radius="${wheel_radius}" material_name="black">
-        <origin xyz='${-base_length*0.5 + wheel_radius} ${-base_length*0.5 + wheel_radius} ${-base_thickness*0.5 - wheel_radius}' rpy='0 0 0'/>
+        <origin xyz="${-base_length*0.5 + wheel_radius} ${-base_length*0.5 + wheel_radius} ${-base_thickness*0.5 - wheel_radius}" rpy="0 0 0"/>
     </xacro:ropod_wheel>
     <xacro:ropod_wheel name="left_front_wheel" parent="base_body" mass="${wheel_mass}"
                        radius="${wheel_radius}" material_name="black">
-        <origin xyz='${base_length*0.5 - wheel_radius} ${base_length*0.5 - wheel_radius} ${-base_thickness*0.5 - wheel_radius}' rpy='0 0 0'/>
+        <origin xyz="${base_length*0.5 - wheel_radius} ${base_length*0.5 - wheel_radius} ${-base_thickness*0.5 - wheel_radius}" rpy="0 0 0"/>
     </xacro:ropod_wheel>
     <xacro:ropod_wheel name="right_front_wheel" parent="base_body" mass="${wheel_mass}"
                        radius="${wheel_radius}" material_name="black">
-        <origin xyz='${base_length*0.5 - wheel_radius} ${-base_length*0.5 + wheel_radius} ${-base_thickness*0.5 - wheel_radius}' rpy='0 0 0'/>
+        <origin xyz="${base_length*0.5 - wheel_radius} ${-base_length*0.5 + wheel_radius} ${-base_thickness*0.5 - wheel_radius}" rpy="0 0 0"/>
     </xacro:ropod_wheel>
     <!-- ======= -->
     <!-- GRIPPER -->
     <!-- ======= -->
-    <joint name='gripper_joint' type='fixed'>
-        <origin xyz='${-base_length*0.5} 0.0 ${wheel_radius*2}' rpy='0 0 0'/>
-        <parent link='base_link'/>
-        <child link='gripper_link'/>
+    <joint name="gripper_joint" type="fixed">
+        <origin xyz="${-base_length*0.5} 0.0 ${wheel_radius*2}" rpy="0 0 0"/>
+        <parent link="base_link"/>
+        <child link="gripper_link"/>
     </joint>
-    <link name='gripper_link'>
+    <link name="gripper_link">
         <visual>
             <geometry>
                 <box size="${0.01} ${0.01} ${0.01}"/>
             </geometry>
-            <origin xyz='0.0 0.0 0.0' rpy='0.0 0.0 0.0' />
+            <origin xyz="0.0 0.0 0.0" rpy="0.0 0.0 0.0" />
             <material name="silver"/>
         </visual>
@@ -119,5 +119,5 @@
                 <box size="${0.01} ${0.01} ${0.01}"/>
             </geometry>
-            <origin xyz='0.0 0.0 0.0' rpy='0.0 0.0 0.0' />
+            <origin xyz="0.0 0.0 0.0" rpy="0.0 0.0 0.0" />
         </collision>
     </link>
@@ -127,5 +127,5 @@
     <xacro:hokuyo name="front_laser" parent="base_body" namespace="${namespace}"
                   ros_topic="scan" update_rate="20" min_angle="-2.36" max_angle="2.36">
-        <origin xyz='0.25 0.0 0.08' rpy='0 0 0'/>
+        <origin xyz="0.25 0.0 0.08" rpy="0 0 0"/>
     </xacro:hokuyo>
     <!-- ====================== -->
@@ -144,13 +144,13 @@
     <!-- DECORATION -->
     <!-- ========== -->
-    <joint name='computer_joint' type='fixed'>
-        <origin xyz='0.0 0.0 0.1' rpy='0 0 0'/>
-        <parent link='base_body_link'/>
-        <child link='computer_link'/>
+    <joint name="computer_joint" type="fixed">
+        <origin xyz="0.0 0.0 0.1" rpy="0 0 0"/>
+        <parent link="base_body_link"/>
+        <child link="computer_link"/>
     </joint>
-    <link name='computer_link'>
+    <link name="computer_link">
         <visual>
             <geometry>
-                <box size='0.2 0.3 0.1'/>
+                <box size="0.2 0.3 0.1"/>
             </geometry>
             <material name="black"/>
@@ -158,5 +158,5 @@
         <collision>
             <geometry>
-                <box size='0.01 0.01 0.01'/>
+                <box size="0.01 0.01 0.01"/>
             </geometry>
         </collision>

Commit message: [mobidik] Changed dimensions based on actual cart measurements

File: description/xacro/mobidik.xacro (robot description, xacro)
@@ -3,9 +3,9 @@
     <xacro:arg name="namespace" default="ropod"/>
     <xacro:property name="namespace" value="$(arg namespace)"/>
-    <xacro:property name="base_length" value="1.1" />
-    <xacro:property name="base_width" value="0.8" />
+    <xacro:property name="base_length" value="0.8" />
+    <xacro:property name="base_width" value="0.72" />
     <xacro:property name="base_thickness" value="0.1" />
-    <xacro:property name="cargo_length" value="1.0" />
-    <xacro:property name="cargo_width" value="0.7" />
+    <xacro:property name="cargo_length" value="0.7" />
+    <xacro:property name="cargo_width" value="0.6" />
     <xacro:property name="cargo_height" value="1.0" />
     <xacro:property name="wheel_radius" value="0.04" />
