Commit message: [description][realsense] Fixed usage of incorrect location of .dae file

File: description/xacro/realsense_d435.xacro (robot description, xacro)
@@ -38,5 +38,5 @@
                 <origin xyz="${d435_cam_mount_from_center_offset} 0.0 ${d435_cam_height/2}" rpy="${pi/2} 0 ${pi/2}"/>
                 <geometry>
-                    <mesh filename="package://kelo_description/meshes/sensors/realsense_d435.dae" />
+                    <mesh filename="package://ropod_sim/description/meshes/realsense_d435.dae" />
                 </geometry>
                 <material name="${name}_aluminum"/>
